Commit message: moveit2 완료

File: rh_plus_7_axis_robot_arm_description/urdf/rh_plus_7_axis_robot_arm.xacro (robot description, xacro)
@@ -208,5 +208,5 @@
 </joint>
 <joint name="Revolute 5" type="revolute">
-  <origin xyz="0.0299 -0.02519 9.1e-05" rpy="0 0 0"/>
+  <origin xyz="0.0299 -0.02519 0.0" rpy="0 0 0"/>
   <parent link="link4"/>
   <child link="link5"/>
@@ -215,5 +215,5 @@
 </joint>
 <joint name="Revolute 6" type="revolute">
-  <origin xyz="0.0611 0.02542 -9.2e-05" rpy="0 0 0"/>
+  <origin xyz="0.0611 0.02542 0.0" rpy="0 0 0"/>
   <parent link="link5"/>
   <child link="gripper_base"/>
@@ -226,5 +226,5 @@
   <child link="gripper_hand_left"/>
   <axis xyz="0.0 -1.0 0.0"/>
-  <limit upper="0.030" lower="0.0" effort="100" velocity="0.015"/>
+  <limit upper="0.030" lower="0.0" effort="100" velocity="0.15"/>
 </joint>
 <joint name="Slider 2" type="prismatic">
@@ -233,5 +233,5 @@
   <child link="gripper_hand_right"/>
   <axis xyz="0.0 1.0 0.0"/>
-  <limit upper="0.030" lower="0.0" effort="100" velocity="0.015"/>
+  <limit upper="0.030" lower="0.0" effort="100" velocity="0.15"/>
   <mimic joint="Slider 1" multiplier="1"/>
 </joint>

Commit message: 조인트 이름변경

File: rh_plus_7_axis_robot_arm_description/urdf/rh_plus_7_axis_robot_arm.xacro (robot description, xacro)
@@ -179,5 +179,5 @@
   </collision>
 </link>
-<joint name="Revolute 1" type="revolute">
+<joint name="revolute_1" type="revolute">
   <origin xyz="0.0 -0.000293 0.045671" rpy="0 0 0"/>
   <parent link="base_link"/>
@@ -186,5 +186,5 @@
   <limit upper="2.094395" lower="-2.094395" effort="100" velocity="5.8178"/>
 </joint>
-<joint name="Revolute 2" type="revolute">
+<joint name="revolute_2" type="revolute">
   <origin xyz="-0.01005 -0.025341 0.021922" rpy="0 0 0"/>
   <parent link="link1"/>
@@ -193,5 +193,5 @@
   <limit upper="1.570796" lower="-1.570796" effort="100" velocity="5.8178"/>
 </joint>
-<joint name="Revolute 3" type="revolute">
+<joint name="revolute_3" type="revolute">
   <origin xyz="0.0 0.000163 0.045" rpy="0 0 0"/>
   <parent link="link2"/>
@@ -200,5 +200,5 @@
   <limit upper="1.658063" lower="-1.570796" effort="100" velocity="5.8178"/>
 </joint>
-<joint name="Revolute 4" type="revolute">
+<joint name="revolute_4" type="revolute">
   <origin xyz="0.0611 0.025492 0.020008" rpy="0 0 0"/>
   <parent link="link3"/>
@@ -207,5 +207,5 @@
   <limit upper="2.094395" lower="-2.094395" effort="100" velocity="5.8178"/>
 </joint>
-<joint name="Revolute 5" type="revolute">
+<joint name="revolute_5" type="revolute">
   <origin xyz="0.0299 -0.02519 0.0" rpy="0 0 0"/>
   <parent link="link4"/>
@@ -214,5 +214,5 @@
   <limit upper="0.698132" lower="-2.094395" effort="100" velocity="5.8178"/>
 </joint>
-<joint name="Revolute 6" type="revolute">
+<joint name="revolute_6" type="revolute">
   <origin xyz="0.0611 0.02542 0.0" rpy="0 0 0"/>
   <parent link="link5"/>
@@ -221,5 +221,5 @@
   <limit upper="2.094395" lower="-2.094395" effort="100" velocity="5.8178"/>
 </joint>
-<joint name="Slider 1" type="prismatic">
+<joint name="slider_1" type="prismatic">
   <origin xyz="0.10160 0.0 0.020148" rpy="0 0 0"/>
   <parent link="gripper_base"/>
@@ -228,5 +228,5 @@
   <limit upper="0.030" lower="0.0" effort="100" velocity="0.15"/>
 </joint>
-<joint name="Slider 2" type="prismatic">
+<joint name="slider_2" type="prismatic">
   <origin xyz="0.10160 0.0 0.020148" rpy="0 0 0"/>
   <parent link="gripper_base"/>
@@ -234,5 +234,5 @@
   <axis xyz="0.0 1.0 0.0"/>
   <limit upper="0.030" lower="0.0" effort="100" velocity="0.15"/>
-  <mimic joint="Slider 1" multiplier="1"/>
+  <mimic joint="slider_1" multiplier="1"/>
 </joint>
 </robot>

File: rh_plus_7_axis_robot_arm_moveit_config/config/rh_plus_7_axis_robot_arm.ros2_control.xacro (robot description, xacro)
@@ -8,50 +8,50 @@
                 <plugin>mock_components/GenericSystem</plugin>
             </hardware>
-            <joint name="Revolute 1">
+            <joint name="revolute_1">
                 <command_interface name="position"/>
                 <state_interface name="position">
-                  <param name="initial_value">${initial_positions['Revolute 1']}</param>
+                  <param name="initial_value">${initial_positions['revolute_1']}</param>
                 </state_interface>
                 <state_interface name="velocity"/>
             </joint>
-            <joint name="Revolute 2">
+            <joint name="revolute_2">
                 <command_interface name="position"/>
                 <state_interface name="position">
-                  <param name="initial_value">${initial_positions['Revolute 2']}</param>
+                  <param name="initial_value">${initial_positions['revolute_2']}</param>
                 </state_interface>
                 <state_interface name="velocity"/>
             </joint>
-            <joint name="Revolute 3">
+            <joint name="revolute_3">
                 <command_interface name="position"/>
                 <state_interface name="position">
-                  <param name="initial_value">${initial_positions['Revolute 3']}</param>
+                  <param name="initial_value">${initial_positions['revolute_3']}</param>
                 </state_interface>
                 <state_interface name="velocity"/>
             </joint>
-            <joint name="Revolute 4">
+            <joint name="revolute_4">
                 <command_interface name="position"/>
                 <state_interface name="position">
-                  <param name="initial_value">${initial_positions['Revolute 4']}</param>
+                  <param name="initial_value">${initial_positions['revolute_4']}</param>
                 </state_interface>
                 <state_interface name="velocity"/>
             </joint>
-            <joint name="Revolute 5">
+            <joint name="revolute_5">
                 <command_interface name="position"/>
                 <state_interface name="position">
-                  <param name="initial_value">${initial_positions['Revolute 5']}</param>
+                  <param name="initial_value">${initial_positions['revolute_5']}</param>
                 </state_interface>
                 <state_interface name="velocity"/>
             </joint>
-            <joint name="Revolute 6">
+            <joint name="revolute_6">
                 <command_interface name="position"/>
                 <state_interface name="position">
-                  <param name="initial_value">${initial_positions['Revolute 6']}</param>
+                  <param name="initial_value">${initial_positions['revolute_6']}</param>
                 </state_interface>
                 <state_interface name="velocity"/>
             </joint>
-            <joint name="Slider 1">
+            <joint name="slider_1">
                 <command_interface name="position"/>
                 <state_interface name="position">
-                  <param name="initial_value">${initial_positions['Slider 1']}</param>
+                  <param name="initial_value">${initial_positions['slider_1']}</param>
                 </state_interface>
                 <state_interface name="velocity"/>

Commit message: 3,5번 서보 방향, 7번 서보 코드 수정

File: rh_plus_7_axis_robot_arm_description/urdf/rh_plus_7_axis_robot_arm.xacro (robot description, xacro)
@@ -197,6 +197,6 @@
   <parent link="link2"/>
   <child link="link3"/>
-  <axis xyz="0.0 -1.0 0.0"/>
-  <limit upper="1.658063" lower="-1.570796" effort="100" velocity="5.8178"/>
+  <axis xyz="0.0 1.0 0.0"/>
+  <limit upper="1.570796" lower="-1.658063" effort="100" velocity="5.8178"/>
 </joint>
 <joint name="revolute_4" type="revolute">
@@ -211,6 +211,6 @@
   <parent link="link4"/>
   <child link="link5"/>
-  <axis xyz="0.0 -1.0 0.0"/>
-  <limit upper="0.698132" lower="-2.094395" effort="100" velocity="5.8178"/>
+  <axis xyz="0.0 1.0 0.0"/>
+  <limit upper="2.094395" lower="-0.698132" effort="100" velocity="5.8178"/>
 </joint>
 <joint name="revolute_6" type="revolute">
@@ -226,5 +226,5 @@
   <child link="gripper_hand_left"/>
   <axis xyz="0.0 -1.0 0.0"/>
-  <limit upper="0.030" lower="0.0" effort="100" velocity="0.15"/>
+  <limit upper="0.030" lower="0.0" effort="100" velocity="0.05"/>
 </joint>
 <joint name="slider_2" type="prismatic">
@@ -233,5 +233,5 @@
   <child link="gripper_hand_right"/>
   <axis xyz="0.0 1.0 0.0"/>
-  <limit upper="0.030" lower="0.0" effort="100" velocity="0.15"/>
+  <limit upper="0.030" lower="0.0" effort="100" velocity="0.05"/>
   <mimic joint="slider_1" multiplier="1"/>
 </joint>
