Commit message: gripper 쪼개서 moveit ball 위치 옮김

File: rh_plus_7_axis_robot_arm_description/urdf/materials.xacro (robot description, xacro)
@@ -19,4 +19,7 @@
   <color rgba="0.361 0.522 0.827 1.000"/>
 </material>
+<material name="pink">
+  <color rgba="1.000 0.412 0.706 1.000"/>
+</material>
 <material name="purple">
   <color rgba="0.690 0.506 0.816 1.000"/>

File: rh_plus_7_axis_robot_arm_description/urdf/rh_plus_7_axis_robot_arm.xacro (robot description, xacro)
@@ -120,9 +120,29 @@
     </collision>
   </link>
+  <link name="link6">
+    <inertial>
+      <origin xyz="0.02193 0.0 0.008597" rpy="0 0 0"/>
+      <mass value="0.076567"/>
+      <inertia ixx="0.0000133" iyy="0.0000256" izz="0.0000179" ixy="0.0" iyz="0.0" ixz="-0.00000175"/>
+    </inertial>
+    <visual>
+      <origin xyz="0 0 0" rpy="0 0 0"/>
+      <geometry>
+        <mesh filename="file://$(find rh_plus_7_axis_robot_arm_description)/meshes/link6.stl" scale="0.001 0.001 0.001"/>
+      </geometry>
+      <material name="pink"/>
+    </visual>
+    <collision>
+      <origin xyz="0 0 0" rpy="0 0 0"/>
+      <geometry>
+        <mesh filename="file://$(find rh_plus_7_axis_robot_arm_description)/meshes/link6.stl" scale="0.001 0.001 0.001"/>
+      </geometry>
+    </collision>
+  </link>
   <link name="gripper_base">
     <inertial>
-      <origin xyz="0.037975 -0.000001 0.015436" rpy="0 0 0"/>
-      <mass value="0.226766"/>
-      <inertia ixx="0.000315358" iyy="0.000079905" izz="0.000337569" ixy="0.000000004" iyz="0.000001911" ixz="-0.000014745"/>
+      <origin xyz="-0.002608 0.0 -0.001469" rpy="0 0 0"/>
+      <mass value="0.124676"/>
+      <inertia ixx="0.0002859" iyy="0.000007381" izz="0.0002819" ixy="0.0" iyz="0.0" ixz="0.0000001069"/>
     </inertial>
     <visual>
@@ -218,10 +238,15 @@
     <origin xyz="0.0611 0.02542 0.0" rpy="0 0 0"/>
     <parent link="link5"/>
-    <child link="gripper_base"/>
+    <child link="link6"/>
     <axis xyz="1.0 0.0 0.0"/>
     <limit upper="2.094395" lower="-2.094395" effort="100" velocity="5.8178"/>
   </joint>
+  <joint name="fixed_1" type="fixed">
+    <origin xyz="0.0464 0.0 0.0201" rpy="0 0 0"/>
+    <parent link="link6"/>
+    <child link="gripper_base"/>
+  </joint>
   <joint name="slider_1" type="prismatic">
-    <origin xyz="0.10160 0.0 0.020148" rpy="0 0 0"/>
+    <origin xyz="0.0552 0.0 0.000048" rpy="0 0 0"/>
     <parent link="gripper_base"/>
     <child link="gripper_hand_left"/>
@@ -230,5 +255,5 @@
   </joint>
   <joint name="slider_2" type="prismatic">
-    <origin xyz="0.10160 0.0 0.020148" rpy="0 0 0"/>
+    <origin xyz="0.0552 0.0 0.000048" rpy="0 0 0"/>
     <parent link="gripper_base"/>
     <child link="gripper_hand_right"/>
