Commit message: 중간 백업

File: rh_plus_7_axis_robot_arm_moveit_config/config/rh_plus_7_axis_robot_arm.ros2_control.xacro (robot description, xacro)
@@ -1,11 +1,16 @@
 <?xml version="1.0"?>
 <robot xmlns:xacro="http://www.ros.org/wiki/xacro">
-    <xacro:macro name="rh_plus_7_axis_robot_arm_ros2_control" params="name initial_positions_file">
+    <xacro:macro name="rh_plus_7_axis_robot_arm_ros2_control" params="name initial_positions_file ros2_control_hardware_type">
         <xacro:property name="initial_positions" value="${xacro.load_yaml(initial_positions_file)['initial_positions']}"/>
         <ros2_control name="${name}" type="system">
             <hardware>
-                <!-- By default, set up controllers for simulation. This won't work on real hardware -->
-                <!-- <plugin>mock_components/GenericSystem</plugin> sa-->
-                <plugin>robotarm_hardware/ROBOTArmSystemHardware</plugin>
+                <xacro:if value="${ros2_control_hardware_type == 'fake'}">
+                    <plugin>mock_components/GenericSystem</plugin>
+                </xacro:if>
+                <xacro:if value="${ros2_control_hardware_type == 'real'}">
+                    <plugin>robotarm_hardware/ROBOTArmSystemHardware</plugin>
+                    <param name="joint_commands_topic">/robotarm_joint_commands</param>
+                    <param name="joint_states_topic">/robotarm_joint_states</param>
+                </xacro:if>
             </hardware>
             <joint name="revolute_1">
@@ -51,11 +56,4 @@
                 <state_interface name="velocity"/>
             </joint>
-            <joint name="slider_1">
-                <command_interface name="position"/>
-                <state_interface name="position">
-                  <param name="initial_value">${initial_positions['slider_1']}</param>
-                </state_interface>
-                <state_interface name="velocity"/>
-            </joint>
         </ros2_control>
     </xacro:macro>

File: rh_plus_7_axis_robot_arm_moveit_config/config/rh_plus_7_axis_robot_arm.urdf.xacro (robot description, xacro)
@@ -2,8 +2,11 @@
 <robot xmlns:xacro="http://www.ros.org/wiki/xacro" name="rh_plus_7_axis_robot_arm">
     <xacro:arg name="initial_positions_file" default="initial_positions.yaml" />
+    <xacro:arg name="ros2_control_hardware_type" default="fake" />
     <!-- Import rh_plus_7_axis_robot_arm urdf file -->
     <xacro:include filename="$(find rh_plus_7_axis_robot_arm_description)/urdf/rh_plus_7_axis_robot_arm.xacro" />
     <!-- Import control_xacro -->
     <xacro:include filename="rh_plus_7_axis_robot_arm.ros2_control.xacro" />
-    <xacro:rh_plus_7_axis_robot_arm_ros2_control name="rh_plus_7_axis_robot_arm" initial_positions_file="$(arg initial_positions_file)"/>
+    <xacro:include filename="rh_plus_7_axis_robot_arm_hand.ros2_control.xacro" />
+    <xacro:rh_plus_7_axis_robot_arm_ros2_control name="RobotarmFakeSystem" initial_positions_file="$(arg initial_positions_file)" ros2_control_hardware_type="$(arg ros2_control_hardware_type)"/>
+    <xacro:rh_plus_7_axis_robot_arm_hand_ros2_control name="RobotarmHandFakeSystem" ros2_control_hardware_type="$(arg ros2_control_hardware_type)"/>
 </robot>

Commit message: 일단 한숨 돌리기

File: rh_plus_7_axis_robot_arm_moveit_config/config/rh_plus_7_axis_robot_arm.ros2_control.xacro (robot description, xacro)
@@ -19,5 +19,7 @@
                   <param name="initial_value">${initial_positions['revolute_1']}</param>
                 </state_interface>
-                <state_interface name="velocity"/>
+                <state_interface name="velocity">
+                    <param name="initial_value">0.0</param>
+                </state_interface>
             </joint>
             <joint name="revolute_2">
@@ -26,5 +28,7 @@
                   <param name="initial_value">${initial_positions['revolute_2']}</param>
                 </state_interface>
-                <state_interface name="velocity"/>
+                <state_interface name="velocity">
+                    <param name="initial_value">0.0</param>
+                </state_interface>
             </joint>
             <joint name="revolute_3">
@@ -33,5 +37,7 @@
                   <param name="initial_value">${initial_positions['revolute_3']}</param>
                 </state_interface>
-                <state_interface name="velocity"/>
+                <state_interface name="velocity">
+                    <param name="initial_value">0.0</param>
+                </state_interface>
             </joint>
             <joint name="revolute_4">
@@ -40,5 +46,7 @@
                   <param name="initial_value">${initial_positions['revolute_4']}</param>
                 </state_interface>
-                <state_interface name="velocity"/>
+                <state_interface name="velocity">
+                    <param name="initial_value">0.0</param>
+                </state_interface>
             </joint>
             <joint name="revolute_5">
@@ -47,5 +55,7 @@
                   <param name="initial_value">${initial_positions['revolute_5']}</param>
                 </state_interface>
-                <state_interface name="velocity"/>
+                <state_interface name="velocity">
+                    <param name="initial_value">0.0</param>
+                </state_interface>
             </joint>
             <joint name="revolute_6">
@@ -54,5 +64,7 @@
                   <param name="initial_value">${initial_positions['revolute_6']}</param>
                 </state_interface>
-                <state_interface name="velocity"/>
+                <state_interface name="velocity">
+                    <param name="initial_value">0.0</param>
+                </state_interface>
             </joint>
         </ros2_control>

File: rh_plus_7_axis_robot_arm_moveit_config/config/rh_plus_7_axis_robot_arm_hand.ros2_control.xacro (robot description, xacro)
@@ -1,6 +1,5 @@
 <?xml version="1.0"?>
 <robot xmlns:xacro="http://www.ros.org/wiki/xacro">
-    <xacro:macro name="rh_plus_7_axis_robot_arm_ros2_control" params="name initial_positions_file ros2_control_hardware_type">
-        <xacro:property name="initial_positions" value="${xacro.load_yaml(initial_positions_file)['initial_positions']}"/>
+    <xacro:macro name="rh_plus_7_axis_robot_arm_hand_ros2_control" params="name ros2_control_hardware_type">
         <ros2_control name="${name}" type="system">
             <hardware>
@@ -17,7 +16,9 @@
                 <command_interface name="position"/>
                 <state_interface name="position">
-                  <param name="initial_value">${initial_positions['slider_1']}</param>
+                  <param name="initial_value">0.0</param>
                 </state_interface>
-                <state_interface name="velocity"/>
+                <state_interface name="velocity">
+                    <param name="initial_value">0.0</param>
+                </state_interface>
             </joint>
         </ros2_control>

Commit message: backup

File: rh_plus_7_axis_robot_arm_moveit_config/config/rh_plus_7_axis_robot_arm.ros2_control.xacro (robot description, xacro)
@@ -15,4 +15,5 @@
                 </xacro:if>
             </hardware>
+            <!--arm-->
             <joint name="revolute_1">
                 <command_interface name="position"/>
@@ -51,4 +52,11 @@
                 </state_interface>
             </joint>
+            <!--hand-->
+            <joint name="slider_1">
+                <command_interface name="position"/>
+                <state_interface name="position">
+                  <param name="initial_value">${initial_positions['slider_1']}</param>
+                </state_interface>
+            </joint>
         </ros2_control>
     </xacro:macro>

File: rh_plus_7_axis_robot_arm_moveit_config/config/rh_plus_7_axis_robot_arm.urdf.xacro (robot description, xacro)
@@ -7,6 +7,4 @@
     <!-- Import control_xacro -->
     <xacro:include filename="rh_plus_7_axis_robot_arm.ros2_control.xacro" />
-    <xacro:include filename="rh_plus_7_axis_robot_arm_hand.ros2_control.xacro" />
     <xacro:rh_plus_7_axis_robot_arm_ros2_control name="RobotarmSystem" initial_positions_file="$(arg initial_positions_file)" ros2_control_hardware_type="$(arg ros2_control_hardware_type)"/>
-    <xacro:rh_plus_7_axis_robot_arm_hand_ros2_control name="RobotarmHandSystem" ros2_control_hardware_type="$(arg ros2_control_hardware_type)"/>
 </robot>
